File: Hardware/loveboard/loveboard.kicad_pcb (KiCad board)
At the start: 2 copper layers, 60.1 x 51.2 mm, 80 parts, among them J1 VCC, J2 BAT, J3 GND, J4 SWCLK, J5 SWDIO, J6 NRST, SW1 SW_SPDT, U1 STM32F40X_LQFP64, U2 BMI160, Y1 8MHz

Commit message: done
Parts:
- added C14: 100n, Capacitor_SMD:C_0603_1608Metric, B.Cu at (179.7, 91.5)
- added H1: ATTCH, MountingHole:MountingHole_2.5mm, F.Cu at (189.9, 87.5)
- moved D6 43.7 mm to (202.5, 92.6), turned to 90 degrees
- moved R6 42.0 mm to (204.1, 92.6), turned to 90 degrees
- moved R7 38.3 mm to (176.0, 92.3), turned to 90 degrees
- moved R20 36.7 mm to (208.8, 83.5), turned to -90 degrees
- moved D7 36.5 mm to (174.4, 92.3), turned to 90 degrees
- moved R18 36.2 mm to (203.2, 83.4), turned to -90 degrees
- moved D18 35.6 mm to (201.6, 83.4), turned to 90 degrees
- moved D20 35.5 mm to (207.2, 83.5), turned to 90 degrees
- moved D3 34.6 mm to (177.2, 84.6), turned to 90 degrees
- moved R3 34.1 mm to (178.9, 84.7), turned to 90 degrees
- moved R4 30.8 mm to (172.9, 84.3), turned to 90 degrees
- moved D4 29.3 mm to (171.2, 84.3), turned to 90 degrees
- moved C1 20.9 mm to (197.9, 95.5), turned to -90 degrees
- moved R19 20.8 mm to (195.6, 112.5), turned to -90 degrees
- moved R13 20.6 mm to (210.2, 94.8), turned to 90 degrees
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Connections:
- U1 pad 61: Net-(U1-Pad61) -> /BMI_INTERRUPT1
- U1 pad 62: /BMI_INTERRUPT -> /BMI_INTERRUPT2
- U2 pad 4: /BMI_INTERRUPT -> /BMI_INTERRUPT1
- U2 pad 9: Net-(U2-Pad9) -> /BMI_INTERRUPT2
Routing:
- net GND: track 0.00 -> 389.2 mm, vias 0 -> 53
- net VCC: track 0.00 -> 181.4 mm, vias 0 -> 9
- net /SWDIO: track 0.00 -> 43.0 mm, vias 0 -> 1
- net /LED_4: track 0.00 -> 39.4 mm, vias 0 -> 2
- net /LED_27: track 0.00 -> 37.5 mm
- net /LED_22: track 0.00 -> 35.7 mm, vias 0 -> 2
- net /LED_3: track 0.00 -> 34.4 mm, vias 0 -> 2
- net /SWCLK: track 0.00 -> 34.3 mm, vias 0 -> 1
- net /LED_21: track 0.00 -> 34.1 mm, vias 0 -> 2
- net /BMI_INTERRUPT1: track 0.00 -> 33.7 mm, vias 0 -> 2
- net /LED_14: track 0.00 -> 29.3 mm, vias 0 -> 2
- net /LED_20: track 0.00 -> 28.9 mm, vias 0 -> 2
- net /NRST: track 0.00 -> 28.7 mm, vias 0 -> 1
- net /LED_12: track 0.00 -> 28.6 mm, vias 0 -> 2
- net /LED_7: track 0.00 -> 28.5 mm, vias 0 -> 2
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- added copper zone on B.Cu, net GND
- added copper zone on F.Cu, net GND
Other:
- outline, holes or cut-outs redrawn
- rule pad_to_mask_clearance: 0.051 -> 0
- board text added: "+3V"
- board text added: "Bo Joel Svensson"
- board text added: "GND"
- board text added: "I love you Andrea!"
- board text added: "NRST"
- board text added: "OFF"
- board text added: "ON"
- board text added: "SWCLK"
- board text added: "SWDIO"
